Commit message: Archivo URDF actualizado

File: Practicas/P01/modelo.urdf (robot description, URDF)
Before this commit: robot rrp_robot, 10 links, 9 joints
Joints:
- joint arm_joint: parent shoulder_link -> armtwo_link; type revolute -> fixed

Commit message: Cambios en el archivo URDF

File: Practicas/P01/modelo.urdf (robot description, URDF)
Before this commit: robot rrp_robot, 10 links, 9 joints
Joints:
- joint arm_joint: origin xyz=0.3 0 0 rpy=0 0 0 -> xyz=-0.05 0.4 0 rpy=0 0 0

Commit message: Archivo final del modelo.urdf

File: Practicas/P01/modelo.urdf (robot description, URDF)
Before this commit: robot rrp_robot, 10 links, 9 joints
Joints:
- joint arm_joint: origin xyz=-0.05 0.4 0 rpy=0 0 0 -> xyz=-0.05 0.4 0 rpy=0 0 3.14

Commit message: Modificacion previa a captura de imagen p1_3.png

File: Practicas/P01/modelo.urdf (robot description, URDF)
Before this commit: robot rrp_robot, 10 links, 9 joints
Joints:
- joint arm_joint: axis 0 0 1 -> (none)
- joint armone_joint: limit (none) -> lower=-1.57 upper=1.57 effort=20.0 velocity=1.0
- joint armtwo_joint: limit (none) -> lower=-1.0 upper=1.0 effort=15.0 velocity=0.8
- joint y_joint: axis 0 0 0 -> (none)
- joint z_joint: axis 0 0 0 -> (none)
